File: mod-sw1.kicad_sch (KiCad schematic)
At the start: 23 parts, among them J1 Conn_01x01_Pin, J11 Conn_01x02_Male, J12 Conn_01x02_Male, J2 Conn_01x01_Pin, J3 Conn_01x01_Pin, J4 Conn_01x01_Pin, J5 G, J6 G, J7 G, J8 G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

Commit message: Add files via upload
Parts:
- C1, C2, C3, C4, C5: value C -> 1000p
- C6: value C -> 0.1u
Other:
- note added: "C1-3 <100M 1000p -> 0.01u J1,3,5 can mount SMA connector M2 screw using TP1,2"
- note added: "SMA"
- company: (none) -> JK1MLY
- title: (none) -> RF SW SKY13453-385LF
Changed lines of the file:
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@@
 (kicad_sch (version 20230121) (generator eeschema)
   (paper "A4")
+  (title_block
+    (title "RF SW SKY13453-385LF")
+    (company "JK1MLY")
+  )
   (junction (at 127 68.58) (diameter 0) (color 0 0 0 0)
   )
@@
   (wire (pts (xy 72.39 57.15) (xy 72.39 54.61))
     (stroke (width 0) (type default))
+  )
+  (text "SMA" (at 62.23 35.56 0)
+    (effects (font (size 1.27 1.27)) (justify left bottom))
+  )
+  (text "C1-3 <100M 1000p -> 0.01u\nJ1,3,5 can mount SMA connector\nM2 screw using TP1,2\n"
+    (at 121.92 25.4 0)
+    (effects (font (size 1.27 1.27)) (justify left bottom))
+  )
+  (text "SMA" (at 205.74 25.4 0)
+    (effects (font (size 1.27 1.27)) (justify left bottom))
+  )
+  (text "SMA" (at 204.47 62.23 0)
+    (effects (font (size 1.27 1.27)) (justify left bottom))
   )
   (symbol (lib_id "RF_Switch:SKY13453-385LF") (at 144.78 59.69 0) (unit 1)
@@
       (effects (font (size 1.27 1.27)))
     )
-    (property "Value" "C" (at 185.42 27.94 90)
+    (property "Value" "1000p" (at 185.42 27.94 90)
       (effects (font (size 1.27 1.27)))
     )
@@
       (effects (font (size 1.27 1.27)))
     )
-    (property "Value" "C" (at 185.42 66.04 90)
+    (property "Value" "1000p" (at 185.42 66.04 90)
       (effects (font (size 1.27 1.27)))
     )
@@
       (effects (font (size 1.27 1.27)) (justify left))
     )
-    (property "Value" "C" (at 119.38 76.835 0)
+    (property "Value" "1000p" (at 119.38 76.835 0)
       (effects (font (size 1.27 1.27)) (justify left))
     )
@@
       (effects (font (size 1.27 1.27)) hide)
     )
-    (property "Datasheet" "~" (at 63.5 45.72 0)
+    (property "Datasheet" "C-13195" (at 63.5 45.72 0)
       (effects (font (size 1.27 1.27)) hide)
     )
@@
       (effects (font (size 1.27 1.27)) (justify left))
     )
-    (property "Value" "C" (at 140.97 76.835 0)
+    (property "Value" "0.1u" (at 140.97 76.835 0)
       (effects (font (size 1.27 1.27)) (justify left))
     )
@@
       (effects (font (size 1.27 1.27)) (justify left))
     )
-    (property "Value" "C" (at 130.81 76.835 0)
+    (property "Value" "1000p" (at 130.81 76.835 0)
       (effects (font (size 1.27 1.27)) (justify left))
     )
@@
       (effects (font (size 1.27 1.27)))
     )
-    (property "Value" "C" (at 120.65 41.91 90)
+    (property "Value" "1000p" (at 120.65 41.91 90)
       (effects (font (size 1.27 1.27)))
     )
@@
       (effects (font (size 1.27 1.27)) hide)
     )
-    (property "Datasheet" "~" (at 205.74 69.85 0)
-      (effects (font (size 1.27 1.27)) hide)
-    )
+    (property "Datasheet" "C-13195" (at 205.74 69.85 0)
+      (effects (font (size 1.27 1.27)) hide)
+    )
